Commit message: feat(biba_hardware_stm32): wire ros2_control SystemInterface end-to-end
Tasks 4-7+10 of epic 6 plan (docs/plans/2026-04-28-biba-hardware-stm32.md).

Task 4 - SystemInterface plugin:
- biba_stm32_system.{hpp,cpp}: BibaStm32SystemHardware (system type)
- Two joints (left_wheel_joint, right_wheel_joint) with velocity command
  and position+velocity state interfaces.
- Open-loop read(): pings STM32 to keep the link alive, reports last
  commanded velocity as state, integrates synthetic position. Wheels
  have no encoders so this matches the physical reality.
- write(): converts diff_drive_controller's rad/s into normalised
  [-1,1] setpoint via the max_wheel_speed hardware param.
- Lifecycle: on_activate opens SPI + ARMs; on_deactivate sends zero
  setpoint and DISARMs; on_shutdown closes transport.
- Hardware params: spi_device, spi_speed_hz, wheel_radius, max_wheel_speed.
- set_link_for_testing() seam for future gtest harness.

Task 5 - pluginlib export:
- biba_hardware_stm32_plugin.xml exporting hardware_interface plugin.
- CMakeLists builds the SHARED lib, target_links biba_stm32_link, runs
  pluginlib_export_plugin_description_file. Build is gated on
  hardware_interface_FOUND so the package still compiles standalone on
  dev machines without ros2_control (gtest path stays green).
- package.xml uncomments the <hardware_interface plugin=...> export.

Task 6 - URDF wiring:
- biba.urdf.xacro: <ros2_control name=BibaSystem type=system> block
  referencing the plugin with spi_device/spi_speed_hz/wheel_radius/
  max_wheel_speed params and the two joints.
- tests/test_biba_description_ros2_control.py: 4 structural tests.

Task 7 - diff_drive_controller config + launch:
- biba_bringup/config/diff_drive_controller.yaml: controller_manager
  declares joint_state_broadcaster + diff_drive_controller; geometry
  mirrors the URDF (wheel_separation=0.30, wheel_radius=0.0425);
  open_loop=true, cmd_vel_timeout=0.5s, linear/angular velocity and
  acceleration limits.
- biba_bringup/launch/control.launch.py: starts robot_state_publisher,
  ros2_control_node, then spawns joint_state_broadcaster and (after it
  exits cleanly) diff_drive_controller.
- tests/test_biba_bringup_control.py: 6 tests (controller types,
  wheel-name/URDF alignment, geometry consistency, open_loop flag,
  launch-file structure).

Task 10 - compose stack swap (also resolves Task 8 architectural
question by killing the Python bridge in composition C):
- docker/ros2/docker-compose.yml: replaced biba-stm32-bridge service
  with biba-control (runs control.launch.py via biba_bringup).
  robot-state-publisher service removed because control.launch.py
  starts RSP itself. /dev/spidev0.0 now has exactly one user.
- docker/ros2/README.md: services table + topics list updated to
  reflect /odom, /joint_states, /tf, /controller_manager/* surface.
- docs/deployment.md: composition C compose table + log command updated.
- scripts/setup/setup_node_ros2.sh and docker/ros2/.env.example:
  dropped BIBA_WHEEL_*/BIBA_*_RATE_HZ/BIBA_CMD_VEL_TIMEOUT_SEC because
  geometry/limits now live in URDF + diff_drive yaml.

Verification:
- colcon build --packages-select biba_hardware_stm32 succeeds locally
  (without ros2_control headers); the SHARED plugin target is silently
  skipped, biba_proto + biba_stm32_link static libs still build, gtest
  passes 12/12.
- pytest: 460 passed (was 450; +10 new structural tests for URDF and
  diff_drive bringup).

File: ros2_ws/src/biba_description/urdf/biba.urdf.xacro (robot description, xacro)
@@ -135,3 +135,39 @@
     <origin xyz="0 0 ${base_height/2.0 + 0.020}" rpy="0 0 0"/>
   </joint>
+  <!-- =================================================================
+       ros2_control hardware interface (composition C).
+       The plugin (biba_hardware_stm32::BibaStm32SystemHardware) owns
+       /dev/spidev0.0 and is the sole user of the STM32 wire protocol.
+       It exposes velocity command + position/velocity state interfaces
+       on the two wheel joints, which diff_drive_controller drives.
+       Hardware parameters:
+         spi_device       — Linux spidev path
+         spi_speed_hz     — SPI clock (1 MHz default; Pi Zero 2W jitter
+                            above ~2 MHz is significant)
+         max_wheel_speed  — wheel angular velocity (rad/s) corresponding
+                            to a normalised setpoint of 1.0; used to
+                            convert diff_drive_controller's rad/s output
+                            into the STM32's normalised wire format
+         wheel_radius     — informational; the controller reads this
+                            from its own yaml, kept here for symmetry
+       ================================================================= -->
+  <ros2_control name="BibaSystem" type="system">
+    <hardware>
+      <plugin>biba_hardware_stm32/BibaStm32SystemHardware</plugin>
+      <param name="spi_device">/dev/spidev0.0</param>
+      <param name="spi_speed_hz">1000000</param>
+      <param name="wheel_radius">${wheel_radius}</param>
+      <param name="max_wheel_speed">20.0</param>
+    </hardware>
+    <joint name="left_wheel_joint">
+      <command_interface name="velocity"/>
+      <state_interface name="position"/>
+      <state_interface name="velocity"/>
+    </joint>
+    <joint name="right_wheel_joint">
+      <command_interface name="velocity"/>
+      <state_interface name="position"/>
+      <state_interface name="velocity"/>
+    </joint>
+  </ros2_control>
 </robot>
