File: kicad/variants/brushed-bts7960/antispark.kicad_sch (KiCad schematic)
At the start: 22 parts, among them J5 SW_ON, Q1 IPB020N10N5, Q2 IPB020N10N5, U8 78L12, U9 LTC7004

Commit message: feat(kicad): измерение тока/напряжения шины и единый выключатель питания (лист 2)
- antispark.kicad_sch: шунт R37 0.5 мОм + INA240A2 (U10) → IBAT, делитель 1:11 → VBAT
- перемычки JP1/JP2 для отключения датчиков с платы в пользу внешнего модуля через H10
- входы U10 разведены Kelvin-дорожками от площадок шунта
- заменён NSD10-48S5 (22–72 В) на NSD10-12S5 (9.8–36 В) — работа на разряженной 6S
- выключатель питания один: J5 (лист 2), вывод SW разъёма J2 отключён (no_connect)
- сервисная перемычка JP3 на цепи SW (R.C./CTRL DC/DC), по умолчанию открыта
- README: обзор найденных решений по счётчику коммутационных пульсаций
Parts:
- added C23, C24: 100n, biba:C0805, symbol Device:C
- added JP1: VBAT c платы, Jumper:SolderJumper-2_P1.3mm_Bridged_RoundedPad1.0x1.5mm, symbol Jumper:SolderJumper_2_Bridged
- added JP2: IBAT c платы, Jumper:SolderJumper-2_P1.3mm_Bridged_RoundedPad1.0x1.5mm, symbol Jumper:SolderJumper_2_Bridged
- added R37: 0.5mR 3W, Resistor_SMD:R_2512_6332Metric, symbol Device:R
- added R38: 100k, biba:R0805, symbol Device:R
- added R39: 10k, biba:R0805, symbol Device:R
- added U10: INA240A2D, Package_SO:SOIC-8_3.9x4.9mm_P1.27mm, symbol Amplifier_Current:INA240A2D
Connections:
- net GND: now also C23.1, C24.1, R39.2, U10.2 (GND), U10.3 (REF2), U10.4 (GND)
- net VIN: now also R37.2, R38.1, U10.1 (-); no longer C19.2, C20.2, Q1.3 (S), Q2.3 (S), R36.1, U9.8 (TS)
- new net: C23.2, JP1.1 (A), R38.2, R39.1
- new net: JP2.1 (A), U10.5
- new net 3.3V: C24.2, U10.6 (V+), U10.7 (REF1)
- new net IBAT: JP2.2 (B)
- new net VBAT: JP1.2 (B)
- new net VSW: C19.2, C20.2, Q1.3 (S), Q2.3 (S), R36.1, R37.1, U10.8 (+), U9.8 (TS)
Other:
- note added: "R37 0.5 мОм → INA240A2 (50 В/В, синфазное −4…+80 В, подавление ШИМ) → 25 мВ/А."
- note added: "REF1=3.3V, REF2=GND → середина 1.65 В, двунаправленно ±66 А (32 мА/LSB)."
- note added: "Антиспарк-выключатель шины 24 В: BAT+ → Q1‖Q2 (N-MOSFET, верхнее плечо) → VSW → шунт R37 → VIN. Драйвер LTC7004, мягкий старт RC на затворе (RG·CG), выключатель — J5."
- note added: "Входы U10 — отдельными (Kelvin) дорожками от площадок R37, не от силовых полигонов."
- note added: "Делитель 100k/10k (1:11): 36 В = 3.3 В. JP1/JP2 замкнуты = VBAT/IBAT с платы;"
- note added: "Измерение шины (как power module APM: шунт + усилитель + делитель):"
- note added: "отрезать, если датчики с внешнего модуля через H10. Прошивка: IBAT 40 А/В,"
- note added: "смещение 1.65 В, BIBA_VBAT_DIVIDER_RATIO ≈ 11 — откалибровать на плате."
- note removed: "Антиспарк-выключатель шины 24 В: BAT+ → Q1‖Q2 (N-MOSFET, верхнее плечо) → VIN. Драйвер LTC7004, мягкий старт RC на затворе (RG·CG), выключатель — J5."
