File: kicad/variants/brushed-bts7960/brushed-bts7960.kicad_pcb (KiCad board)
At the start: 2 copper layers, 180.3 x 100.1 mm, 494 parts, among them IC1 rp2040_RP2040_breakout_swd, J1 HDR-M-2.54_1x3, J2 HDR-M-2.54_1x4, J3 HDR-M-2.54_1x4, J4 HDR-M-2.54_1x4, U1 SN74AHC244DW, U2 BTN7970, U3 BTN7970, U4 BTN7970, U5 BTN7970, U6 BMI160, U7 SPX3819M5-L-3-3/TR

Commit message: feat(kicad): перенос силовых клемм, DC/DC и антиспарка на плату + скрипт Update PCB from Schematic
Parts:
- removed PM2: NSD10-48S5, Converter_DCDC_MeanWell_NSD10_THT
- removed Pad_gge6729: Pad_gge6729, Pad_gge6729
- removed Pad_gge6765: Pad_gge6765, Pad_gge6765
- removed Pad_gge6789: Pad_gge6789, Pad_gge6789
- removed Pad_gge6813: Pad_gge6813, Pad_gge6813
- removed Pad_gge6837: Pad_gge6837, Pad_gge6837
- removed Pad_gge6861: Pad_gge6861, Pad_gge6861
- added C17: 1u 50V, biba:C0805, F.Cu at (238.9, 142.2)
- added C18: 10n, biba:C0805, F.Cu at (211.3, 142.4)
- added C19: 470n 100V, Capacitor_SMD:C_1206_3216Metric, F.Cu at (223.9, 142.2)
- added C20: 10u 25V, Capacitor_SMD:C_1206_3216Metric, F.Cu at (240.0, 137.0)
- added C21: 100n, biba:C0805, F.Cu at (217.1, 147.1)
- added C22: 1u, biba:C0805, F.Cu at (214.8, 147.1)
- added C23: 100n, biba:C0805, F.Cu at (230.9, 147.1)
- added C24: 100n, biba:C0805, F.Cu at (236.5, 137.0)
- added D3: 27V, Diode_SMD:D_SMA, F.Cu at (233.9, 142.2)
- added D4: BAS116, Diode_SMD:D_SOD-123, F.Cu at (215.0, 142.2)
- added D5: LED зел., LED_SMD:LED_0805_2012Metric, F.Cu at (241.6, 147.1)
- added J5: SW_ON, Connector_PinHeader_2.54mm:PinHeader_1x02_P2.54mm_Vertical, F.Cu at (213.0, 135.8)
- added J6: RIPPLE, Connector_PinHeader_2.54mm:PinHeader_1x14_P2.54mm_Vertical, F.Cu at (92.3, 100.0)
- added J7: M1, biba:WirePad_1x2_P7.62mm_D2.0mm, F.Cu at (266.8, 59.0)
- added J8: M2, biba:WirePad_1x2_P7.62mm_D2.0mm, F.Cu at (266.8, 99.5)
- added J9: BAT, biba:WirePad_1x2_P7.62mm_D2.0mm, F.Cu at (266.8, 131.0)
- added JP1: VBAT c платы, Jumper:SolderJumper-2_P1.3mm_Bridged_RoundedPad1.0x1.5mm, F.Cu at (234.4, 147.1)
- added JP2: IBAT c платы, Jumper:SolderJumper-2_P1.3mm_Bridged_RoundedPad1.0x1.5mm, F.Cu at (237.9, 147.1)
- added JP3: DC/DC OFF (сервис), Jumper:SolderJumper-2_P1.3mm_Open_RoundedPad1.0x1.5mm, F.Cu at (140.0, 54.5)
- added JP4: IS_L→ADC, Jumper:SolderJumper-2_P1.3mm_Bridged_RoundedPad1.0x1.5mm, F.Cu at (102.4, 118.8)
- added JP5: IS_R→ADC, Jumper:SolderJumper-2_P1.3mm_Bridged_RoundedPad1.0x1.5mm, F.Cu at (103.3, 116.3)
- added Q1: IPB020N10N5, Package_TO_SOT_SMD:TO-263-2, F.Cu at (256.0, 132.1)
- added Q2: IPB020N10N5, Package_TO_SOT_SMD:TO-263-2, F.Cu at (256.0, 143.6)
- added R29: 10R, biba:R0805, F.Cu at (226.8, 142.2)
- added R30: 10R, biba:R0805, F.Cu at (229.1, 142.2)
- added R31: 100k, biba:R0805, F.Cu at (218.8, 142.2)
- added R32: 10R, biba:R0805, F.Cu at (221.1, 142.2)
- added R33: 100R, Resistor_SMD:R_1206_3216Metric, F.Cu at (212.0, 147.1)
- added R34: 100k, biba:R0805, F.Cu at (219.4, 147.1)
- added R35: 22k, biba:R0805, F.Cu at (221.7, 147.1)
- added R36: 6.8k, biba:R0805, F.Cu at (224.0, 147.1)
- added R37: 0.5mR 3W, Resistor_SMD:R_2512_6332Metric, F.Cu at (239.5, 131.5)
- added R38: 100k, biba:R0805, F.Cu at (226.3, 147.1)
- added R39: 10k, biba:R0805, F.Cu at (228.6, 147.1)
- added U10: INA240A2D, Package_SO:SOIC-8_3.9x4.9mm_P1.27mm, F.Cu at (231.5, 137.0)
- added U8: 78L12, Package_TO_SOT_SMD:SOT-89-3, F.Cu at (224.5, 137.0)
- added U9: LTC7004, Package_SO:MSOP-10-1EP_3x3mm_P0.5mm_EP1.68x1.88mm, F.Cu at (218.5, 137.0)
- C10, C11, C12, C13: footprint C0805 -> biba:C0805
- C14: footprint CAP-TH_BD16.0-P7.50-D0.8-FD-H25.0 -> biba:CAP-TH_BD16.0-P7.50-D0.8-FD-H25.0
- C15, C16: footprint C_Rect_L10.0mm_W5.0mm_P5.00mm_P7.50mm -> Capacitor_THT:C_Rect_L10.0mm_W5.0mm_P5.00mm_P7.50mm
- D1, D2: footprint D_DO-201AE_P15.24mm_Horizontal -> Diode_THT:D_DO-201AE_P15.24mm_Horizontal
- PM1: value SKMW30f-05 -> SKMW30G-05 / NSD10-12S5; footprint biba:SKMW30G-05 -> biba:DCDC_SKMW30_NSD10
- R27, R28: footprint R_Axial_Power_L25.0mm_W9.0mm_P30.48mm -> Resistor_THT:R_Axial_Power_L25.0mm_W9.0mm_P30.48mm
- moved PM1 87.4 mm to (248.0, 70.5), turned to 0 degrees
- moved C15 2.00 mm to (234.0, 82.5)
- moved C16 2.00 mm to (234.0, 118.5)
- moved R27 2.00 mm to (226.0, 54.0)
- moved R28 2.00 mm to (226.0, 90.0)
Connections:
- net IC1_34 renamed Net-(IC1-GP28)
- net IC1_35 renamed Net-(IC1-GP29)
- net M1_SNUB renamed /M1_SNUB
- net M2_SNUB renamed /M2_SNUB
- net PM1_4 renamed Net-(PM1-TRIM)
- net U2_5 renamed Net-(U2-SR)
- net U2_6 renamed Net-(U2-IS)
- net U3_5 renamed Net-(U3-SR)
- net U3_6 renamed Net-(U3-IS)
- net U4_5 renamed Net-(U4-SR)
- net U4_6 renamed Net-(U4-IS)
- net U5_5 renamed Net-(U5-SR)
- net U5_6 renamed Net-(U5-IS)
- net U6_12 renamed Net-(U6-CSB)
- IC1 pad 30: (no net) -> unconnected-(IC1-RUN-Pad30)
- IC1 pad 31: R_IS -> ADC_R
- IC1 pad 32: L_IS -> ADC_L
- IC1 pad 36: (no net) -> unconnected-(IC1-3V3-Pad36)
- IC1 pad 37: (no net) -> unconnected-(IC1-GP23-Pad37)
- IC1 pad 40: (no net) -> unconnected-(IC1-Vout-Pad40)
- IC1 pad 41: (no net) -> unconnected-(IC1-3V3-Pad41)
- IC1 pad 42: (no net) -> unconnected-(IC1-SWDIO-Pad42)
- IC1 pad 43: (no net) -> unconnected-(IC1-SWDCLK-Pad43)
- J2 pad 1: SW -> unconnected-(J2-Pad1)
- U6 pad 10: (no net) -> unconnected-(U6-OCSB-Pad10)
- U6 pad 11: (no net) -> unconnected-(U6-OSDO-Pad11)
- U6 pad 2: (no net) -> unconnected-(U6-ASDX-Pad2)
- U6 pad 3: (no net) -> unconnected-(U6-ASCX-Pad3)
- U6 pad 9: (no net) -> unconnected-(U6-INT2-Pad9)
- U7 pad 4: (no net) -> unconnected-(U7-BYP-Pad4)
Routing:
- net +5V: track 269.0 -> 502.2 mm, vias 0 -> 1
- net Net-(PM1-TRIM): track 9.67 -> 210.0 mm, vias 0 -> 1
- net GND: track 338.2 -> 226.2 mm, vias 22 -> 23
- net SW: track 48.0 -> 146.8 mm, vias 0 -> 1
- net M2-: track 88.0 -> 176.4 mm
- net M1+: track 55.2 -> 128.1 mm
- net M2+: track 65.0 -> 124.3 mm
- net M1-: track 73.3 -> 132.5 mm
- net VIN: track 246.1 -> 278.9 mm, vias 0 -> 1
- net VSW: track 0.00 -> 24.6 mm
- net BAT+: track 0.00 -> 18.8 mm
- net R_IS: track 81.2 -> 76.5 mm
- net L_IS: track 81.6 -> 77.8 mm
- net ADC_R: track 0.00 -> 3.35 mm
- net ADC_L: track 0.00 -> 2.46 mm
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Other:
- board text removed: "BAT"
- board text removed: "M1"
- board text removed: "M2"
